File: pcb/aurora_l.kicad_pcb (KiCad board)
At the start: 2 copper layers, 118 x 114.2 mm, 89 parts

Commit message: Refine left board further
Parts:
- added ?: , , F.Cu at (103.6, 102.6)
- added ?: , , F.Cu at (42.9, 196.1)
- added ?: , , F.Cu at (139.6, 111.1)
Changed lines of the file:
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@@
 		)
 	)
+	(footprint ""
+		(layer "F.Cu")
+		(at 103.6 102.6)
+		(property "Reference" ""
+			(at 0 0 0)
+			(layer "F.SilkS")
+			(effects
+				(font
+					(size 1.27 1.27)
+					(thickness 0.15)
+				)
+			)
+		)
+		(property "Value" ""
+			(at 0 0 0)
+			(layer "F.Fab")
+			(effects
+				(font
+					(size 1.27 1.27)
+					(thickness 0.15)
+				)
+			)
+		)
+		(property "Footprint" ""
+			(at 0 0 0)
+			(layer "F.Fab")
+			(hide yes)
+			(effects
+				(font
+					(size 1.27 1.27)
+					(thickness 0.15)
+				)
+			)
+		)
+		(property "Datasheet" ""
+			(at 0 0 0)
+			(layer "F.Fab")
+			(hide yes)
+			(effects
+				(font
+					(size 1.27 1.27)
+					(thickness 0.15)
+				)
+			)
+		)
+		(property "Description" ""
+			(at 0 0 0)
+			(layer "F.Fab")
+			(hide yes)
+			(effects
+				(font
+					(size 1.27 1.27)
+					(thickness 0.15)
+				)
+			)
+		)
+		(pad "" np_thru_hole circle
+			(at 0 0 90)
+			(size 4 4)
+			(drill 4)
+			(layers "*.Cu" "*.Mask" "F.SilkS")
+			(clearance 0.3)
+		)
+	)
 	(footprint "ComboDiode"
 		(layer "F.Cu")
@@
 		)
 	)
+	(footprint ""
+		(layer "F.Cu")
+		(at 42.85 196.1)
+		(property "Reference" ""
+			(at 0 0 0)
+			(layer "F.SilkS")
+			(effects
+				(font
+					(size 1.27 1.27)
+					(thickness 0.15)
+				)
+			)
+		)
+		(property "Value" ""
+			(at 0 0 0)
+			(layer "F.Fab")
+			(effects
+				(font
+					(size 1.27 1.27)
+					(thickness 0.15)
+				)
+			)
+		)
+		(property "Footprint" ""
+			(at 0 0 0)
+			(layer "F.Fab")
+			(hide yes)
+			(effects
+				(font
+					(size 1.27 1.27)
+					(thickness 0.15)
+				)
+			)
+		)
+		(property "Datasheet" ""
+			(at 0 0 0)
+			(layer "F.Fab")
+			(hide yes)
+			(effects
+				(font
+					(size 1.27 1.27)
+					(thickness 0.15)
+				)
+			)
+		)
+		(property "Description" ""
+			(at 0 0 0)
+			(layer "F.Fab")
+			(hide yes)
+			(effects
+				(font
+					(size 1.27 1.27)
+					(thickness 0.15)
+				)
+			)
+		)
+		(pad "" np_thru_hole circle
+			(at 0 0 90)
+			(size 4 4)
+			(drill 4)
+			(layers "*.Cu" "*.Mask" "F.SilkS")
+			(clearance 0.3)
+		)
+	)
 	(footprint "WS2812-2020"
 		(layer "F.Cu")
@@
 		)
 	)
+	(footprint ""
+		(layer "F.Cu")
+		(at 139.6 111.1)
+		(property "Reference" ""
+			(at 0 0 0)
+			(layer "F.SilkS")
+			(effects
+				(font
+					(size 1.27 1.27)
+					(thickness 0.15)
+				)
+			)
+		)
+		(property "Value" ""
+			(at 0 0 0)
+			(layer "F.Fab")
+			(effects
+				(font
+					(size 1.27 1.27)
+					(thickness 0.15)
+				)
+			)
+		)
+		(property "Footprint" ""
+			(at 0 0 0)
+			(layer "F.Fab")
+			(hide yes)
+			(effects
+				(font
+					(size 1.27 1.27)
+					(thickness 0.15)
+				)
+			)
+		)
+		(property "Datasheet" ""
+			(at 0 0 0)
+			(layer "F.Fab")
+			(hide yes)
+			(effects
+				(font
+					(size 1.27 1.27)
+					(thickness 0.15)
+				)
+			)
+		)
+		(property "Description" ""
+			(at 0 0 0)
+			(layer "F.Fab")
+			(hide yes)
+			(effects
+				(font
+					(size 1.27 1.27)
+					(thickness 0.15)
+				)
+			)
+		)
+		(pad "" np_thru_hole circle
+			(at 0 0 90)
+			(size 4 4)
+			(drill 4)
+			(layers "*.Cu" "*.Mask" "F.SilkS")
+			(clearance 0.3)
+		)
+	)
 	(footprint "ComboDiode"
 		(layer "F.Cu")
@@
 	)
 	(segment
-		(start 135.5 158.81)
-		(end 135.5 114)
+		(start 135.5 114)
+		(end 135.5 158.81)
 		(width 0.25)
 		(layer "B.Cu")
@@
 	)
 	(segment
-		(start 126.105 104.605)
-		(end 70.855 104.605)
+		(start 135.5 158.81)
+		(end 141.19 164.5)
 		(width 0.25)
 		(layer "B.Cu")
@@
 	)
 	(segment
-		(start 135.5 114)
-		(end 126.105 104.605)
+		(start 73.75 107.5)
+		(end 129 107.5)
 		(width 0.25)
 		(layer "B.Cu")
@@
 	)
 	(segment
-		(start 123.19 164.5)
-		(end 125.35 164.5)
+		(start 129 107.5)
+		(end 135.5 114)
 		(width 0.25)
 		(layer "B.Cu")
@@
 	)
 	(segment
-		(start 70.855 104.605)
-		(end 61.51 95.26)
+		(start 61.51 95.26)
+		(end 73.75 107.5)
 		(width 0.25)
 		(layer "B.Cu")
@@
 	)
 	(segment
-		(start 141.19 164.5)
-		(end 135.5 158.81)
+		(start 123.19 164.5)
+		(end 125.35 164.5)
 		(width 0.25)
 		(layer "B.Cu")
