File: ergogen/output/pcbs/aurora_r.kicad_pcb (KiCad board)
At the start: 2 copper layers, 182.9 x 101.4 mm, 121 parts

Commit message: Organize pins and clean up led footprint
Connections:
- net P011 renamed P03
- net P029 renamed P10
- net P031 renamed P09
- net P100 renamed P04
- net P104 renamed P02
- net P106 renamed P01
- net P113 renamed P13
- net P115 renamed P12
- D17 pad 1: P002 -> P11
- D18 pad 1: P002 -> P11
- D19 pad 1: P002 -> P11
- D20 pad 1: P002 -> P11
- D21 pad 1: P002 -> P11
- D22 pad 1: P002 -> P11
- D23 pad 1: P002 -> P11
- REF** pad 1: VCC -> P010 (x38)
- REF** pad 2: P010 -> VCC (x38)
- REF** pad 3: GND -> P009 (x38)
- REF** pad 4: P009 -> GND (x38)
- S10 pad 2: P024 -> P05
- S11 pad 2: P022 -> P06
- S12 pad 2: P022 -> P06
- S13 pad 2: P020 -> P07
- S14 pad 2: P020 -> P07
- S15 pad 2: P017 -> P08
- S16 pad 2: P017 -> P08
- S21 pad 2: P024 -> P05
- S22 pad 2: P022 -> P06
- S23 pad 2: P020 -> P07
- S28 pad 2: P024 -> P05
- S29 pad 2: P022 -> P06
- S30 pad 2: P020 -> P07
- S31 pad 2: P017 -> P08
- S36 pad 2: P022 -> P05
- S37 pad 2: P020 -> P06
- S38 pad 2: P017 -> P07
- S9 pad 2: P024 -> P05

Commit message: Simplify LED rotations
Parts:
- turned REF** to 0 degrees (x15)
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